File: RP_port_tester_v0.kicad_sch (KiCad schematic)
At the start: 0 parts

Commit message: Initial Schematic and component selection
Parts:
- added C1, C10, C11, C12, C13, C14, C19, C21, C22, C4, C5, C8, C9: 100n, Capacitor_SMD:C_0603_1608Metric_Pad1.08x0.95mm_HandSolder, symbol Device:C
- added C15, C16: 15p, Capacitor_SMD:C_0402_1005Metric_Pad0.74x0.62mm_HandSolder, symbol Device:C_Small
- added C17, C3: 22u, Capacitor_SMD:C_1206_3216Metric_Pad1.33x1.80mm_HandSolder, symbol Device:C
- added C18, C6, C7: 1u, Capacitor_SMD:C_0603_1608Metric_Pad1.08x0.95mm_HandSolder, symbol Device:C
- added C2: 10u, Capacitor_SMD:C_1206_3216Metric_Pad1.33x1.80mm_HandSolder, symbol Device:C
- added C20: 2n2, Capacitor_SMD:C_0402_1005Metric_Pad0.74x0.62mm_HandSolder, symbol Device:C
- added D1, D2: GREEN, Diode_SMD:D_0805_2012Metric_Pad1.15x1.40mm_HandSolder, symbol Device:LED
- added D10, D4, D6, D8: GREEN, LED_THT:LED_D3.0mm, symbol Device:LED
- added D3, D5, D7, D9: YELLOW, LED_THT:LED_D3.0mm, symbol Device:LED
- added J1: USB_B PORT0, My_Library:USB_B_Vertical, symbol Connector:USB_B
- added J2: USB_B PORT1, My_Library:USB_B_Vertical, symbol Connector:USB_B
- added J3: USB_B PORT2, My_Library:USB_B_Vertical, symbol Connector:USB_B
- added J4: USB_B PORT3, My_Library:USB_B_Vertical, symbol Connector:USB_B
- added J5, J6, J7, J8: DE9_Pins, My_Library:DB9_Horizontal, symbol Connector:DE9_Pins
- added J9: UART, Connector_PinHeader_2.54mm:PinHeader_1x03_P2.54mm_Vertical, symbol Connector:Conn_01x03_Pin
- added LS1: ABI-001-RC, Buzzer_Beeper:Buzzer_15x7.5RM7.6, symbol Device:Speaker_Crystal
- added Q1: IRLZ44N, Package_TO_SOT_THT:TO-220-3_Vertical, symbol Transistor_FET:IRLZ44N
- added R1: DNF, Resistor_SMD:R_0603_1608Metric_Pad0.98x0.95mm_HandSolder, symbol Device:R
- added R10, R12, R6, R8: 220R, Resistor_SMD:R_0603_1608Metric_Pad0.98x0.95mm_HandSolder, symbol Device:R
- added R11, R13, R5, R7, R9: 390R, Resistor_SMD:R_0603_1608Metric_Pad0.98x0.95mm_HandSolder, symbol Device:R
- added R14, R3: 27R4, Resistor_SMD:R_0603_1608Metric_Pad0.98x0.95mm_HandSolder, symbol Device:R
- added R15, R18, R2, R21, R23, R24: 1k, Resistor_SMD:R_0603_1608Metric_Pad0.98x0.95mm_HandSolder, symbol Device:R
- added R16: 70k, Resistor_SMD:R_0603_1608Metric_Pad0.98x0.95mm_HandSolder, symbol Device:R
- added R17, R22: 100k, Resistor_SMD:R_0603_1608Metric_Pad0.98x0.95mm_HandSolder, symbol Device:R
- added R19: 12k, Resistor_SMD:R_0603_1608Metric_Pad0.98x0.95mm_HandSolder, symbol Device:R
- added R20, R29: 100R, Resistor_SMD:R_0603_1608Metric_Pad0.98x0.95mm_HandSolder, symbol Device:R
- added R25: 47R, Resistor_SMD:R_0603_1608Metric_Pad0.98x0.95mm_HandSolder, symbol Device:R
- added R26: 120k, Resistor_SMD:R_0603_1608Metric_Pad0.98x0.95mm_HandSolder, symbol Device:R
- added R27: 0R51, Resistor_THT:R_Axial_DIN0309_L9.0mm_D3.2mm_P15.24mm_Horizontal, symbol Device:R
- added R28: 10k, Resistor_SMD:R_0603_1608Metric_Pad0.98x0.95mm_HandSolder, symbol Device:R
- added R4: 180R, Resistor_SMD:R_0603_1608Metric_Pad0.98x0.95mm_HandSolder, symbol Device:R
- added SW1: BOOTSEL, Button_Switch_SMD:SW_SPST_PTS645Sx43SMTR92, symbol Switch:SW_Push
- added U1: AMS1117-3.3, Package_TO_SOT_SMD:SOT-223-3_TabPin2, symbol Regulator_Linear:AMS1117-3.3
- added U2, U3, U6: STMPS2151, Package_TO_SOT_SMD:SOT-23-5_HandSoldering, symbol My_Library:STMPS2151STR
- added U4: FSUSB74MPX, Package_DFN_QFN:QFN-16-1EP_3x3mm_P0.5mm_EP1.7x1.7mm_ThermalVias, symbol My_Library:FSUSB74MPX
- added U5: W25Q128JVS, Package_SO:SOIC-8_5.3x5.3mm_P1.27mm, symbol Memory_Flash:W25Q128JVS
- added U7: RP2040, Package_DFN_QFN:QFN-56-1EP_7x7mm_P0.4mm_EP3.2x3.2mm_ThermalVias, symbol MCU_RaspberryPi:RP2040
- added U8: LM2904, Package_DIP:DIP-8_W7.62mm, symbol Amplifier_Operational:LM2904
- added Y1: ABM8-272-T3, Crystal:Crystal_SMD_Abracon_ABM8G-4Pin_3.2x2.5mm, symbol Device:Crystal_GND24
Connections:
- new net: D2.1 (K), R5.1
- new net: Q1.3 (S), R23.1, R25.2, R27.1
- new net: C21.1, R23.2, U8.5 (+)
- new net: R26.1, R28.1, U8.6 (-)
- new net: R24.1, R26.2, U8.7
- new net: C20.1, R20.1, U8.1
- new net: Q1.1 (G), R20.2, R22.2
- new net: C20.2, R25.1, U8.2 (-)
- new net: D5.1 (K), R8.1
- new net: LS1.1, R29.2
- new net: R2.2, SW1.1
- new net: D6.1 (K), R9.1
- new net: D1.1 (K), R4.1
- new net: D3.1 (K), R6.1
- new net: D7.1 (K), R10.1
- new net: C19.1, R19.2, R21.1, U8.3 (+)
- new net: D10.1 (K), R13.1
- new net: C15.2, U7.20 (XIN), Y1.1
- new net: C16.2, R15.1, Y1.3
- new net: C18.1, R18.2, R19.1
- new net: D4.1 (K), R7.1
- new net: D9.1 (K), R12.1
- new net: J6.2, J6.3
- new net: J8.2, J8.3
- new net: D8.1 (K), R11.1
- new net: R15.2, U7.21 (XOUT)
- new net: J7.2, J7.3
- new net: J5.2, J5.3
- new net +1V1: C4.1, C5.1, C6.1, U7.23 (DVDD), U7.45 (VREG_VOUT), U7.50 (DVDD)
- new net +3.3V: C1.1, C10.1, C11.1, C12.1, C13.1, C14.1, C3.1, C7.1, C8.1, C9.1, D1.2 (A), R1.1, U1.2 (VO), U4.4 (VCC), U5.8 (VCC), U7.1 (IOVDD), U7.10 (IOVDD), U7.22 (IOVDD), U7.33 (IOVDD), U7.42 (IOVDD), U7.43 (ADC_AVDD), U7.44 (VREG_IN), U7.48 (USB_VDD), U7.49 (IOVDD)
- new net GND: C1.2, C10.2, C11.2, C12.2, C13.2, C14.2, C15.1, C16.1, C17.2, C18.2, C19.2, C2.2, C21.2, C22.2, C3.2, C4.2, C5.2, C6.2, C7.2, C8.2, C9.2, J1.4 (GND), J2.4 (GND), J3.4 (GND), J4.4 (GND), J9.1 (Pin_1), LS1.2, R10.2, R11.2, R12.2, R13.2, R17.2, R21.2, R22.1, R27.2, R28.2, R4.2, R5.2, R6.2, R7.2, R8.2, R9.2, SW1.2, U1.1 (GND), U2.2 (GND), U3.2 (GND), U4.1 (GND), U4.15 (~{OE}), U4.17 (PAD), U5.4 (GND), U6.2 (GND), U7.19 (TESTEN), U7.57 (GND), U8.4 (V-), Y1.2, Y1.4
- new net PICO_AUDIO_EN: R29.1, U7.35 (GPIO23)
- new net PICO_CURRENT_ADC: C22.1, R24.2, U7.39 (GPIO27_ADC1)
- new net PICO_LOAD_PWM: R18.1, U7.8 (GPIO6)
- new net PICO_PORT0_TESTED: D4.2 (A), U7.29 (GPIO18)
- new net PICO_PORT1_TESTED: D6.2 (A), U7.30 (GPIO19)
- new net PICO_PORT2_TESTED: D8.2 (A), U7.31 (GPIO20)
- new net PICO_PORT3_TESTED: D10.2 (A), U7.32 (GPIO21)
- new net PICO_USB_D+: R14.1, U4.2 (D+)
- new net PICO_USB_D-: R3.1, U4.3 (D-)
- new net PICO_VBUS_ADC: R16.2, R17.1, U7.38 (GPIO26_ADC0)
- new net QSPI_SCLK: U5.6 (CLK), U7.52 (QSPI_SCLK)
- new net QSPI_SD0: U5.5 (DI/IO_{0}), U7.53 (QSPI_SD0)
- new net QSPI_SD1: U5.2 (DO/IO_{1}), U7.55 (QSPI_SD1)
- new net QSPI_SD2: U5.3 (~{WP}/IO_{2}), U7.54 (QSPI_SD2)
- new net QSPI_SD3: U5.7 (~{HOLD}/~{RESET}/IO_{3}), U7.51 (QSPI_SD3)
- new net QSPI_SS: R1.2, R2.1, U5.1 (~{CS}), U7.56 (QSPI_SS)
- new net UART_RX: J9.2 (Pin_2), U7.3 (GPIO1)
- new net UART_TX: J9.3 (Pin_3), U7.2 (GPIO0)
- new net USB0_D+: J1.3 (D+), U4.13 (HSD0+)
- new net USB0_D-: J1.2 (D-), U4.14 (HSD0-)
- new net USB1_D+: J2.3 (D+), U4.11 (HSD1+)
- new net USB1_D-: J2.2 (D-), U4.12 (HSD1-)
- new net USB1_VBUS: D5.2 (A), J2.1 (VBUS), U2.5 (IN)
- new net USB1_VBUS_EN: U2.4 (EN), U7.12 (GPIO9)
- new net USB2_D+: J3.3 (D+), U4.10 (HSD2+)
- new net USB2_D-: J3.2 (D-), U4.9 (HSD2-)
- new net USB2_VBUS: D7.2 (A), J3.1 (VBUS), U3.5 (IN)
- new net USB2_VBUS_EN: U3.4 (EN), U7.13 (GPIO10)
- new net USB3_D+: J4.3 (D+), U4.8 (HSD3+)
- new net USB3_D-: J4.2 (D-), U4.7 (HSD3-)
- new net USB3_VBUS: D9.2 (A), J4.1 (VBUS), U6.5 (IN)
- new net USB3_VBUS_EN: U6.4 (EN), U7.14 (GPIO11)
- new net USBMUX_SEL0: U4.6 (SEL0), U7.16 (GPIO13)
- new net USBMUX_SEL1: U4.5 (SEL1), U7.17 (GPIO14)
- new net USB_DN: R14.2, U7.46 (USB_DM)
- new net USB_DP: R3.2, U7.47 (USB_DP)
- new net VBUS: C2.1, D3.2 (A), J1.1 (VBUS), U1.3 (VI), U8.8 (V+)
- new net VBUS_TEST: C17.1, D2.2 (A), Q1.2 (D), R16.1, U2.1 (OUT), U3.1 (OUT), U6.1 (OUT)
- no-connect marks 0 -> 39
Other:
- note added: "Buzzer"
- note added: "DB9 Loopback Connectors"
- note added: "Flash Memory"
- note added: "Microcontroller"
- note added: "Per port LED indicators"
- note added: "Power"
- note added: "Programmable VBUS Load"
- note added: "RC-Filter"
- note added: "SMD Status LEDs"
- note added: "Status LEDs"
- note added: "UART Connector"
- note added: "USB Connectors"
- note added: "USB MUX"
- note added: "VBUS Switches"
- note added: "VBUS Voltage Div"
- note added: "Voltage Div 0-3.3V -> 0-250mV"

Commit message: Layout and Tracing
Parts:
- removed D10, D4, D6, D8: GREEN, LED_THT:LED_D3.0mm, symbol Device:LED
- removed D3, D5, D7, D9: YELLOW, LED_THT:LED_D3.0mm, symbol Device:LED
- removed J1: USB_B PORT0, My_Library:USB_B_Vertical, symbol Connector:USB_B
- removed J2: USB_B PORT1, My_Library:USB_B_Vertical, symbol Connector:USB_B
- removed J3: USB_B PORT2, My_Library:USB_B_Vertical, symbol Connector:USB_B
- removed J4: USB_B PORT3, My_Library:USB_B_Vertical, symbol Connector:USB_B
- removed R10, R12, R6, R8: 220R, Resistor_SMD:R_0603_1608Metric_Pad0.98x0.95mm_HandSolder, symbol Device:R
- removed R11, R13, R7, R9: 390R, Resistor_SMD:R_0603_1608Metric_Pad0.98x0.95mm_HandSolder, symbol Device:R
- removed U2, U3, U6: STMPS2151, Package_TO_SOT_SMD:SOT-23-5_HandSoldering, symbol My_Library:STMPS2151STR
- added C23: 100n, Capacitor_SMD:C_0603_1608Metric_Pad1.08x0.95mm_HandSolder, symbol Device:C
- added FID1, FID2, FID3, FID4, FID5: Fiducial, Fiducial:Fiducial_1mm_Mask2mm, symbol Mechanical:Fiducial
- added H1, H3, H5: TOOLING_HOLE, MountingHole:ToolingHole_1.152mm, symbol Mechanical:MountingHole
- added H2, H4, H6: MountingHole, MountingHole:MountingHole_3.2mm_M3, symbol Mechanical:MountingHole
- added TP1, TP2, TP3, TP4: TestPoint, TestPoint:TestPoint_Plated_Hole_D2.0mm, symbol Connector:TestPoint
- Q1: footprint Package_TO_SOT_THT:TO-220-3_Vertical -> Package_TO_SOT_THT:TO-220-3_Horizontal_TabDown
- renumbered J5 to J1, J6 to J2, J7 to J3, J8 to J4, J9 to J5, R18 to R10, R19 to R11, R20 to R12, R21 to R13, R22 to R14, R23 to R15, R24 to R16, R25 to R17, R26 to R18, R27 to R19, R28 to R20, R29 to R21, R14 to R4, R4 to R5, R5 to R6, R15 to R7, R16 to R8, R17 to R9, U5 to U2, U4 to U3, U7 to U4, U8 to U5
Connections:
- net +3.3V: now also TP2.1
- net GND: now also C23.2, TP4.1
- net PICO_AUDIO_EN: now also U4.7 (GPIO5); no longer U4.35 (GPIO23)
- net PICO_LOAD_PWM: now also U4.5 (GPIO3); no longer U4.8 (GPIO6)
- net PICO_USB_D+: now also R3.1; no longer R4.1
- net PICO_USB_D-: now also R4.1; no longer R3.1
- net PICO_VBUS_ADC: now also C23.1
- net USB1_VBUS_EN: now also U4.14 (GPIO11); no longer U4.12 (GPIO9)
- net USB3_VBUS_EN: now also U4.12 (GPIO9); no longer U4.14 (GPIO11)
- net VBUS: now also TP1.1
- net VBUS_TEST: now also TP3.1
- net Shunt High: now reaches Q1.3 (S), R15.1, R17.2, R19.1
- net Amp Gain+: now reaches C21.1, R15.2, U5.5 (+)
- net Amp Gain-: now reaches R18.1, R20.1, U5.6 (-)
- net Amp Gain Out: now reaches R16.1, R18.2, U5.7
- net Amp Current Out: now reaches C20.1, R12.1, U5.1
- net FET-Gate: now reaches Q1.1 (G), R12.2, R14.2
- net Amp Current-: now reaches C20.2, R17.1, U5.2 (-)
- net BOOTSEL_BTN: now reaches R2.2, SW1.1
- net Amp Current+: now reaches C19.1, R11.2, R13.1, U5.3 (+)
- net PICO_XIN: now reaches C15.2, U4.20 (XIN), Y1.1
- net Crystal_Out: now reaches C16.2, R7.1, Y1.3
- net PWM_Filt: now reaches C18.1, R10.2, R11.1
- net PICO_XOUT: now reaches R7.2, U4.21 (XOUT)
- no-connect marks 39 -> 32
Other:
- added sheet USB Connectors (usb.kicad_sch)
- note added: "Holes & Fiducials"
- note added: "Test Points"
- note removed: "Per port LED indicators"
- note removed: "Status LEDs"
- note removed: "USB Connectors"
- note removed: "VBUS Switches"
- moved on the sheet: C15, C16, C18, C19, C20, C22, D1, D2, LS1, R10, R11, R13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

Commit message: Final layout and routing
Parts:
- C1, C10, C11, C12, C13, C14, C19, C21, C22, C23, C4, C5, C8, C9: value 100n -> 100nF
- C15, C16: value 15p -> 15pF
- C17, C3: value 22u -> 22uF
- C18, C6, C7: value 1u -> 1uF
- C2: value 10u -> 10uF
- C20: value 2n2 -> 2.2nF
- J1, J2, J3, J4, J5, LS1, Q1, R19, SW1, U5: now left out of the parts list
- R5: value 180R -> 220R
- R8: value 70k -> 68k
Connections:
- no-connect marks 32 -> 46
Changed lines of the file:
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@@
 	)
 	(no_connect
+		(at 113.03 167.64)
+	)
+	(no_connect
 		(at 41.91 271.78)
 	)
@@
 	)
 	(no_connect
+		(at 113.03 127)
+	)
+	(no_connect
+		(at 113.03 172.72)
+	)
+	(no_connect
+		(at 113.03 121.92)
+	)
+	(no_connect
 		(at 69.85 271.78)
 	)
@@
 	)
 	(no_connect
+		(at 113.03 170.18)
+	)
+	(no_connect
 		(at 69.85 254)
 	)
@@
 	)
 	(no_connect
+		(at 113.03 149.86)
+	)
+	(no_connect
+		(at 113.03 154.94)
+	)
+	(no_connect
 		(at 41.91 232.41)
 	)
@@
 	)
 	(no_connect
+		(at 113.03 152.4)
+	)
+	(no_connect
 		(at 69.85 237.49)
 	)
@@
 	)
 	(no_connect
+		(at 62.23 111.76)
+	)
+	(no_connect
 		(at 41.91 224.79)
 	)
@@
 	)
 	(no_connect
+		(at 113.03 116.84)
+	)
+	(no_connect
 		(at 41.91 266.7)
 	)
 	(no_connect
+		(at 113.03 175.26)
+	)
+	(no_connect
+		(at 113.03 142.24)
+	)
+	(no_connect
 		(at 41.91 274.32)
 	)
@@
 	)
 	(no_connect
+		(at 113.03 129.54)
+	)
+	(no_connect
 		(at 62.23 177.8)
 	)
@@
 	)
 	(no_connect
+		(at 113.03 132.08)
+	)
+	(no_connect
 		(at 69.85 242.57)
 	)
@@
 		(unit 1)
 		(exclude_from_sim no)
-		(in_bom yes)
+		(in_bom no)
 		(on_board yes)
 		(dnp no)
@@
 		(unit 2)
 		(exclude_from_sim no)
-		(in_bom yes)
+		(in_bom no)
 		(on_board yes)
 		(dnp no)
@@
 			)
 		)
-		(property "Value" "100n"
+		(property "Value" "100nF"
 			(at 189.23 95.2499 0)
 			(effects
@@
 			)
 		)
-		(property "Value" "2n2"
+		(property "Value" "2.2nF"
 			(at 292.1 215.8999 0)
 			(effects
@@
 		(unit 3)
 		(exclude_from_sim no)
-		(in_bom yes)
+		(in_bom no)
 		(on_board yes)
 		(dnp no)
@@
 		(unit 1)
 		(exclude_from_sim no)
-		(in_bom yes)
+		(in_bom no)
 		(on_board yes)
 		(dnp no)
@@
 		(unit 1)
 		(exclude_from_sim no)
-		(in_bom yes)
+		(in_bom no)
 		(on_board yes)
 		(dnp no)
@@
 			)
 		)
-		(property "Value" "180R"
+		(property "Value" "220R"
 			(at 364.49 128.2699 0)
 			(effects
@@
 			)
 		)
-		(property "Value" "100n"
+		(property "Value" "100nF"
 			(at 392.43 227.3299 0)
 			(effects
@@
 			)
 		)
-		(property "Value" "100n"
+		(property "Value" "100nF"
 			(at 143.51 95.2499 0)
 			(effects
@@
 			)
 		)
-		(property "Value" "100n"
+		(property "Value" "100nF"
 			(at 120.65 95.2499 0)
 			(effects
@@
 		(unit 1)
 		(exclude_from_sim no)
-		(in_bom yes)
+		(in_bom no)
 		(on_board yes)
 		(dnp no)
@@
 			)
 		)
-		(property "Value" "100n"
+		(property "Value" "100nF"
 			(at 166.37 95.2499 0)
 			(effects
@@
 			)
 		)
-		(property "Value" "70k"
+		(property "Value" "68k"
 			(at 375.92 177.7999 0)
 			(effects
@@
 		(unit 1)
 		(exclude_from_sim no)
-		(in_bom yes)
+		(in_bom no)
 		(on_board yes)
 		(dnp no)
@@
 			)
 		)
-		(property "Value" "22u"
+		(property "Value" "22uF"
 			(at 365.76 177.7999 0)
 			(effects
@@
 			)
 		)
-		(property "Value" "100n"
+		(property "Value" "100nF"
 			(at 339.09 224.7899 0)
 			(effects
@@
 			)
 		)
-		(property "Value" "1u"
+		(property "Value" "1uF"
 			(at 224.79 209.5499 0)
 			(effects
@@
 		(unit 1)
 		(exclude_from_sim no)
-		(in_bom yes)
+		(in_bom no)
 		(on_board yes)
 		(dnp no)
@@
 			)
 		)
-		(property "Value" "100n"
+		(property "Value" "100nF"
 			(at 132.08 95.2499 0)
 			(effects
@@
 		(unit 1)
 		(exclude_from_sim no)
-		(in_bom yes)
+		(in_bom no)
 		(on_board yes)
 		(dnp no)
@@
 			)
 		)
-		(property "Value" "100n"
+		(property "Value" "100nF"
 			(at 257.81 209.5499 0)
 			(effects
@@
 			)
 		)
-		(property "Value" "100n"
+		(property "Value" "100nF"
 			(at 63.5 95.2499 0)
 			(effects
@@
 			)
 		)
-		(property "Value" "10u"
+		(property "Value" "10uF"
 			(at 33.02 39.3699 0)
 			(effects
@@
 			)
 		)
-		(property "Value" "15p"
+		(property "Value" "15pF"
 			(at 21.5963 153.67 90)
 			(effects
@@
 			)
 		)
-		(property "Value" "15p"
+		(property "Value" "15pF"
 			(at 21.59 173.99 90)
 			(effects
@@
 			)
 		)
-		(property "Value" "100n"
+		(property "Value" "100nF"
 			(at 177.8 95.2499 0)
 			(effects
@@
 			)
 		)
-		(property "Value" "22u"
+		(property "Value" "22uF"
 			(at 57.15 39.3699 0)
 			(effects
@@
 			)
 		)
-		(property "Value" "100n"
+		(property "Value" "100nF"
 			(at 154.94 95.2499 0)
 			(effects
@@
 			)
 		)
-		(property "Value" "100n"
+		(property "Value" "100nF"
 			(at 388.62 187.9599 0)
 			(effects
@@
 			)
 		)
-		(property "Value" "100n"
+		(property "Value" "100nF"
 			(at 106.68 31.7499 0)
 			(effects
@@
 			)
 		)
-		(property "Value" "1u"
+		(property "Value" "1uF"
 			(at 76.2 95.2499 0)
 			(effects
@@
 		(unit 1)
 		(exclude_from_sim no)
-		(in_bom yes)
+		(in_bom no)
 		(on_board yes)
 		(dnp no)
@@
 		(unit 1)
 		(exclude_from_sim no)
-		(in_bom yes)
+		(in_bom no)
 		(on_board yes)
 		(dnp no)
@@
 			)
 		)
-		(property "Value" "100n"
+		(property "Value" "100nF"
 			(at 50.8 95.2499 0)
 			(effects
@@
 		(unit 1)
 		(exclude_from_sim no)
-		(in_bom yes)
+		(in_bom no)
 		(on_board yes)
 		(dnp no)
@@
 			)
 		)
-		(property "Value" "1u"
+		(property "Value" "1uF"
 			(at 111.76 95.2499 0)
 			(effects
